File: final-project/Obstacle_detector/Obstacle_detector.kicad_sch (KiCad schematic)
At the start: 12 parts, among them U1 SeeeduinoXIAO, U2 VL53L8CXV0GC/1, U3 TCA9544A, U4 VL53L8CXV0GC/1, U5 TLV73318PDBV

Commit message: Updated final project
Parts:
- R6, R7: value 10kΩ -> 4.7kΩ
Connections:
- net +1V8: now also U2.B7 (CORE_1V8), U4.B7 (CORE_1V8); no longer U2.A3 (IOVDD), U4.A3 (IOVDD)
- net +3.3V: now also R6.2, R7.2; no longer R6.1, R7.1
- net GND: now also U1.13 (GND), U3.1 (A0), U3.2 (A1), U3.3 (A2); no longer U1.16 (GND)
- net at U1.5 (PA8_A4_D4_SDA), U3.19 (SDA): now also R6.1
- net at U1.6 (PA9_A5_D5_SCL), U3.18 (SCL): now also R7.1
- now unconnected: U1.2 (PA4_A1_D1), U1.3 (PA10_A2_D2)
- no-connect marks 43 -> 44
